Commit message: Basic multi-launcable mirtes

File: urdf/mirte_master_description.autogen.urdf (robot description, URDF)
Before this commit: robot mirtebot_description, 11 links, 10 joints
Links:
- link base_link: geometry collision mesh filename=package://mirte_master_simulator/meshes/base_link.STL; visual mesh filename=package://mirte_master_simulator/meshes/base_link.STL
- link camera_link: geometry collision mesh filename=package://mirte_master_simulator/meshes/camera_link.STL; visual mesh filename=package://mirte_master_simulator/meshes/camera_link.STL
- link fron_left_ultrasone_link: geometry collision mesh filename=package://mirte_master_simulator/meshes/fron_left_ultrasone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; visual mesh filename=package://mirte_master_simulator/meshes/fron_left_ultrasone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
- link fron_right_ultrasone_link: geometry collision mesh filename=package://mirte_master_simulator/meshes/fron_right_ultrason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; visual mesh filename=package://mirte_master_simulator/meshes/fron_right_ultrason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
- link front_left_wheel_link: geometry collision mesh filename=package://mirte_master_simulator/meshes/front_left_wheel_li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; visual mesh filename=package://mirte_master_simulator/meshes/front_left_wheel_li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
- link front_right_wheel_link: geometry collision mesh filename=package://mirte_master_simulator/meshes/front_right_wheel_l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; visual mesh filename=package://mirte_master_simulator/meshes/front_right_wheel_l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
- link lidar_link: geometry collision mesh filename=package://mirte_master_simulator/meshes/lidar_link.STL; visual mesh filename=package://mirte_master_simulator/meshes/lidar_link.STL
- link rear_left_ultrasone_link: geometry collision mesh filename=package://mirte_master_simulator/meshes/rear_left_ultrasone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; visual mesh filename=package://mirte_master_simulator/meshes/rear_left_ultrasone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
- link rear_left_wheel_link: geometry collision mesh filename=package://mirte_master_simulator/meshes/rear_left_wheel_lin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; visual mesh filename=package://mirte_master_simulator/meshes/rear_left_wheel_lin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
- link rear_right_ultrasone_link: geometry collision mesh filename=package://mirte_master_simulator/meshes/rear_right_ultrason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; visual mesh filename=package://mirte_master_simulator/meshes/rear_right_ultrason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
- link rear_right_wheel_link: geometry collision mesh filename=package://mirte_master_simulator/meshes/rear_right_wheel_li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; visual mesh filename=package://mirte_master_simulator/meshes/rear_right_wheel_li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
