Commit message: Initial Attempt at open Gazebo Drivable based on zm_robot

File: urdf/mirte_master_description.urdf.xacro (robot description, xacro)
@@ -5,7 +5,17 @@
      For more information, please see http://wiki.ros.org/sw_urdf_exporter -->
 <robot
-  name="mirte_master">
-  <link
-    name="base_link">
+  name="mirte_master" xmlns:xacro="http://ros.org/wiki/xacro">
+  <!-- Bring in simulation data for Gazebo. -->
+  <xacro:include filename="$(find mirte_master_simulator)/urdf/mirte_master_description.gazebo" />
+  <!-- Add Pseudo link to fix warning about intertia on startup -->
+  <link name="base_link"></link>
+  <joint name="bl_bb_joint" type="fixed">
+    <parent
+      link="base_link" />
+    <child
+      link="base_body" />
+  </joint>
+  <link
+    name="base_body">
     <inertial>
       <origin
@@ -78,9 +88,8 @@
     <collision>
       <origin
-        xyz="0 0 0"
-        rpy="0 0 0" />
-      <geometry>
-        <mesh
-          filename="package://mirte_master_simulator/meshes/front_left_wheel_link.STL" />
+        xyz="0.030103 0.034202 0.03996"
+        rpy="0 0 0" />
+      <geometry>
+        <cylinder radius="0.053" length="0.06"/>
       </geometry>
     </collision>
@@ -88,14 +97,14 @@
   <joint
     name="front_left_wheel_joint"
-    type="fixed">
+    type="continuous">
     <origin
       xyz="0.16802 -0.050672 -0.07546"
       rpy="1.5708 0.13151 -1.5708" />
-    <parent
-      link="base_link" />
+      <parent
+      link="base_body" />
     <child
       link="front_left_wheel_link" />
     <axis
-      xyz="0 0 0" />
+      xyz="0 0 -1" />
   </joint>
   <link
@@ -131,9 +140,8 @@
     <collision>
       <origin
-        xyz="0 0 0"
-        rpy="0 0 0" />
-      <geometry>
-        <mesh
-          filename="package://mirte_master_simulator/meshes/front_right_wheel_link.STL" />
+        xyz="0.030103 0.034202 0.03996"
+        rpy="0 0 0" />
+      <geometry>
+        <cylinder radius="0.053" length="0.06"/>
       </geometry>
     </collision>
@@ -141,14 +149,14 @@
   <joint
     name="front_right_wheel_joint"
-    type="fixed">
+    type="continuous">
     <origin
       xyz="-0.087976 -0.060085 -0.083647"
       rpy="1.5708 -0.14316 -1.5708" />
     <parent
-      link="base_link" />
+      link="base_body" />
     <child
       link="front_right_wheel_link" />
     <axis
-      xyz="0 0 0" />
+      xyz="0 0 1" />
   </joint>
   <link
@@ -184,9 +192,8 @@
     <collision>
       <origin
-        xyz="0 0 0"
-        rpy="0 0 0" />
-      <geometry>
-        <mesh
-          filename="package://mirte_master_simulator/meshes/rear_right_wheel_link.STL" />
+        xyz="0.030103 0.034202 0.03996"
+        rpy="0 0 0" />
+      <geometry>
+        <cylinder radius="0.053" length="0.06"/>
       </geometry>
     </collision>
@@ -194,14 +201,14 @@
   <joint
     name="rear_right_wheel_joint"
-    type="fixed">
+    type="continuous">
     <origin
       xyz="-0.087976 0.11997 -0.074702"
       rpy="1.5708 0.15337 -1.5708" />
     <parent
-      link="base_link" />
+      link="base_body" />
     <child
       link="rear_right_wheel_link" />
     <axis
-      xyz="0 0 0" />
+      xyz="0 0 1" />
   </joint>
   <link
@@ -237,9 +244,8 @@
     <collision>
       <origin
-        xyz="0 0 0"
-        rpy="0 0 0" />
-      <geometry>
-        <mesh
-          filename="package://mirte_master_simulator/meshes/rear_left_wheel_link.STL" />
+        xyz="0.030103 0.034202 0.03996"
+        rpy="0 0 0" />
+      <geometry>
+        <cylinder radius="0.053" length="0.06"/>
       </geometry>
     </collision>
@@ -247,14 +253,14 @@
   <joint
     name="rear_left_wheel_joint"
-    type="fixed">
+    type="continuous">
     <origin
       xyz="0.16802 0.10992 -0.083647"
       rpy="1.5708 -0.14316 -1.5708" />
     <parent
-      link="base_link" />
+      link="base_body" />
     <child
       link="rear_left_wheel_link" />
     <axis
-      xyz="0 0 0" />
+      xyz="0 0 -1" />
   </joint>
   <link
@@ -305,5 +311,5 @@
       rpy="1.5708 0 0" />
     <parent
-      link="base_link" />
+      link="base_body" />
     <child
       link="camera_link" />
@@ -358,5 +364,5 @@
       rpy="-1.5708 0 -1.5708" />
     <parent
-      link="base_link" />
+      link="base_body" />
     <child
       link="lidar_link" />
@@ -411,5 +417,5 @@
       rpy="3.1416 0 0.29671" />
     <parent
-      link="base_link" />
+      link="base_body" />
     <child
       link="fron_left_ultrasone_link" />
@@ -464,5 +470,5 @@
       rpy="3.1416 0 -0.29671" />
     <parent
-      link="base_link" />
+      link="base_body" />
     <child
       link="fron_right_ultrasone_link" />
@@ -517,5 +523,5 @@
       rpy="3.1416 0 2.8449" />
     <parent
-      link="base_link" />
+      link="base_body" />
     <child
       link="rear_left_ultrasone_link" />
@@ -570,5 +576,5 @@
       rpy="3.14159265358979 0 -2.84488668075076" />
     <parent
-      link="base_link" />
+      link="base_body" />
     <child
       link="rear_right_ultrasone_link" />
